Commit message: corrected stl names

File: src/mecapkg/urdf/mecabot.urdf.xacro (robot description, xacro)
@@ -55,19 +55,19 @@
       <geometry>
         <mesh
-          filename="file://$(find mecapkg)/meshes/chassis.STL" />
-      </geometry>
-      <material
-        name="">
-        <color
-          rgba="0.79216 0.81961 0.93333 1" />
-      </material>
-    </visual>
-    <collision>
-      <origin
-        xyz="0 0 0"
-        rpy="0 0 0" />
-      <geometry>
-        <mesh
-          filename="file://$(find mecapkg)/meshes/chassis.STL" />
+          filename="file://$(find mecapkg)/meshes/chassis.stl" />
+      </geometry>
+      <material
+        name="">
+        <color
+          rgba="0.79216 0.81961 0.93333 1" />
+      </material>
+    </visual>
+    <collision>
+      <origin
+        xyz="0 0 0"
+        rpy="0 0 0" />
+      <geometry>
+        <mesh
+          filename="file://$(find mecapkg)/meshes/chassis.stl" />
       </geometry>
     </collision>
@@ -95,19 +95,19 @@
       <geometry>
         <mesh
-          filename="file://$(find mecapkg)/meshes/fl.STL" />
-      </geometry>
-      <material
-        name="">
-        <color
-          rgba="0.79216 0.81961 0.93333 1" />
-      </material>
-    </visual>
-    <collision>
-      <origin
-        xyz="0 0 0"
-        rpy="0 0 0" />
-      <geometry>
-        <mesh
-          filename="file://$(find mecapkg)/meshes/fl.STL" />
+          filename="file://$(find mecapkg)/meshes/fl.stl" />
+      </geometry>
+      <material
+        name="">
+        <color
+          rgba="0.79216 0.81961 0.93333 1" />
+      </material>
+    </visual>
+    <collision>
+      <origin
+        xyz="0 0 0"
+        rpy="0 0 0" />
+      <geometry>
+        <mesh
+          filename="file://$(find mecapkg)/meshes/fl.stl" />
       </geometry>
     </collision>
@@ -148,19 +148,19 @@
       <geometry>
         <mesh
-          filename="file://$(find mecapkg)/meshes/br.STL" />
-      </geometry>
-      <material
-        name="">
-        <color
-          rgba="0.79216 0.81961 0.93333 1" />
-      </material>
-    </visual>
-    <collision>
-      <origin
-        xyz="0 0 0"
-        rpy="0 0 0" />
-      <geometry>
-        <mesh
-          filename="file://$(find mecapkg)/meshes/br.STL" />
+          filename="file://$(find mecapkg)/meshes/br.stl" />
+      </geometry>
+      <material
+        name="">
+        <color
+          rgba="0.79216 0.81961 0.93333 1" />
+      </material>
+    </visual>
+    <collision>
+      <origin
+        xyz="0 0 0"
+        rpy="0 0 0" />
+      <geometry>
+        <mesh
+          filename="file://$(find mecapkg)/meshes/br.stl" />
       </geometry>
     </collision>
@@ -201,19 +201,19 @@
       <geometry>
         <mesh
-          filename="file://$(find mecapkg)/meshes/fr.STL" />
-      </geometry>
-      <material
-        name="">
-        <color
-          rgba="0.79216 0.81961 0.93333 1" />
-      </material>
-    </visual>
-    <collision>
-      <origin
-        xyz="0 0 0"
-        rpy="0 0 0" />
-      <geometry>
-        <mesh
-          filename="file://$(find mecapkg)/meshes/fr.STL" />
+          filename="file://$(find mecapkg)/meshes/fr.stl" />
+      </geometry>
+      <material
+        name="">
+        <color
+          rgba="0.79216 0.81961 0.93333 1" />
+      </material>
+    </visual>
+    <collision>
+      <origin
+        xyz="0 0 0"
+        rpy="0 0 0" />
+      <geometry>
+        <mesh
+          filename="file://$(find mecapkg)/meshes/fr.stl" />
       </geometry>
     </collision>
@@ -254,19 +254,19 @@
       <geometry>
         <mesh
-          filename="file://$(find mecapkg)/meshes/bl.STL" />
-      </geometry>
-      <material
-        name="">
-        <color
-          rgba="0.79216 0.81961 0.93333 1" />
-      </material>
-    </visual>
-    <collision>
-      <origin
-        xyz="0 0 0"
-        rpy="0 0 0" />
-      <geometry>
-        <mesh
-          filename="file://$(find mecapkg)/meshes/bl.STL" />
+          filename="file://$(find mecapkg)/meshes/bl.stl" />
+      </geometry>
+      <material
+        name="">
+        <color
+          rgba="0.79216 0.81961 0.93333 1" />
+      </material>
+    </visual>
+    <collision>
+      <origin
+        xyz="0 0 0"
+        rpy="0 0 0" />
+      <geometry>
+        <mesh
+          filename="file://$(find mecapkg)/meshes/bl.stl" />
       </geometry>
     </collision>
